Commit message: first commit

File: urdf/realrobot.urdf.xacro (robot description, xacro)
@@ -6,11 +6,11 @@
         <parent link="base_footprint"/>
         <child link="base_link"/>
-        <origin xyz="0.0 0.0 0.10" rpy="0 0 0"/>
+        <origin xyz="0.0 0.0 0.055" rpy="0 0 0"/>
     </joint>
     <link name="base_link">
         <visual>
-            <origin xyz="0 0 0.04" rpy="0.0 0.0 0.0" />
-            <geometry>
-                <box size="0.5 0.3 0.08"/>
+            <origin xyz="0 0 0.03" rpy="0.0 0.0 0.0" />
+            <geometry>
+                <box size="0.255 0.15 0.06"/>
             </geometry>
             <material name="blue">
@@ -19,7 +19,7 @@
         </visual>
         <collision>
-            <origin xyz="0 0 0.12" rpy="0.0 0.0 0.0" />
-            <geometry>
-                <box size="0.5 0.3 0.08"/>
+            <origin xyz="0 0 0.03" rpy="0.0 0.0 0.0" />
+            <geometry>
+                <box size="0.255 0.15 0.06"/>
             </geometry>
         </collision>
@@ -32,17 +32,17 @@
         <parent link="base_link"/>
         <child link="caster_back_link"/>
-        <origin xyz="-0.18 0 0" rpy="0 0 0"/>
+        <origin xyz="-0.08 0 0" rpy="0 0 0"/>
     </joint>
     <link name="caster_back_link">
         <visual name="caster">
-            <origin xyz="0.0 0 -0.05"/>
-            <geometry>
-                <sphere radius="0.05"/>
-            </geometry>
-        </visual>
-        <collision>
-          <origin xyz="0 0 -0.05" />
+            <origin xyz="0.0 0 -0.0275"/>
+            <geometry>
+                <sphere radius="0.0275"/>
+            </geometry>
+        </visual>
+        <collision>
+          <origin xyz="0 0 -0.0275" />
           <geometry>
-            <sphere radius="0.05"/>
+            <sphere radius="0.0275"/>
           </geometry>
         </collision>
@@ -58,5 +58,5 @@
         <parent link="base_link"/>
         <child link="right_wheel"/>
-        <origin xyz="0.1 -0.185 0.0" rpy="-1.570795 0 0"/>
+        <origin xyz="0.08 -0.0875 -0.0225" rpy="-1.570795 0 0"/>
         <axis xyz="0.0 0 1"/>
     </joint>
@@ -64,5 +64,5 @@
         <visual>
             <geometry>
-                <cylinder radius="0.1" length="0.07"/>
+                <cylinder radius="0.0325" length="0.025"/>
             </geometry>
             <material name="black">
@@ -72,5 +72,5 @@
         <collision>
             <geometry>
-                <cylinder radius="0.1" length="0.07"/>
+                <cylinder radius="0.0325" length="0.025"/>
             </geometry>
         </collision>
@@ -84,5 +84,5 @@
         <parent link="base_link"/>
         <child link="left_wheel"/>
-        <origin xyz="0.1 0.185 0.0" rpy="-1.570795 0 0"/>
+        <origin xyz="0.08 0.0875 -0.0225" rpy="-1.570795 0 0"/>
         <axis xyz="0.0 0 1"/>
     </joint>
@@ -90,5 +90,5 @@
         <visual>
             <geometry>
-                <cylinder radius="0.1" length="0.07"/>
+                <cylinder radius="0.0325" length="0.025"/>
             </geometry>
             <material name="black">
@@ -98,5 +98,5 @@
         <collision>
             <geometry>
-                <cylinder radius="0.1" length="0.07"/>
+                <cylinder radius="0.0325" length="0.025"/>
             </geometry>
         </collision>
@@ -107,4 +107,5 @@
         </inertial>
     </link>
+ <!--
     <joint name="cylinder1_" type="fixed">
         <parent link="base_link"/>
@@ -294,14 +295,15 @@
         </inertial>
     </link>
+-->
     <joint name="joint_laser" type="fixed">
         <parent link="base_link"/>
-        <child link="laser_frame"/>
-        <origin xyz="-0.18 0 0.26" rpy="0 0 0"/>
-    </joint>
-    <link name="laser_frame">
-        <visual>
-            <origin xyz="0 0 0.02" rpy="0 0 0"/>
-            <geometry>
-                <cylinder radius="0.03" length="0.04"/>
+        <child link="laser"/>
+        <origin xyz="0.08 0 0.085" rpy="0 0 -3.1415"/>
+    </joint>
+    <link name="laser">
+        <visual>
+            <origin xyz="0 0 0.0" rpy="0 0 0"/>
+            <geometry>
+                <cylinder radius="0.035" length="0.05"/>
             </geometry>
             <material name="orange">
@@ -311,7 +313,28 @@
         <collision>
             <geometry>
+                <cylinder radius="0.035" length="0.05"/>
+            </geometry>
+        </collision>
+    </link>
+    <!-- <joint name="joint_imu" type="fixed">
+        <parent link="base_link"/>
+        <child link="imu_link"/>
+        <origin xyz="-0.14 0 0.26" rpy="0 0 0"/>
+    </joint>
+    <link name="imu_link">
+        <visual>
+            <origin xyz="0 0 0.02" rpy="0 0 0"/>
+            <geometry>
                 <cylinder radius="0.03" length="0.04"/>
             </geometry>
-        </collision>
-    </link>
+            <material name="orange">
+                <color rgba="0.1 0.5 0.05 1"/>
+            </material>
+        </visual>
+        <collision>
+            <geometry>
+                <cylinder radius="0.03" length="0.04"/>
+            </geometry>
+        </collision>
+    </link>  -->
 </robot>
